Commit message: 调整joint2/3/4关节限位 (URDF + MuJoCo)

File: robotic_sldasm_ros2_humble/urdf/robotic_sldasm.urdf (robot description, URDF)
Before this commit: robot robotic_sldasm, 5 links, 4 joints
Joints:
- joint joint2: limit lower=-1.57079632679 upper=1.57079632679 effort=10.0 velocity=2.0 -> lower=0 upper=3.14159265359 effort=10.0 velocity=2.0
- joint joint3: limit lower=-1.57079632679 upper=1.57079632679 effort=10.0 velocity=2.0 -> lower=-2.51327412287 upper=2.51327412287 effort=10.0 velocity=2.0
- joint joint4: limit lower=-1.57079632679 upper=1.57079632679 effort=10.0 velocity=2.0 -> lower=-2.09439510239 upper=2.09439510239 effort=10.0 velocity=2.0
