Commit message: 目录重组 + robotic_description 描述包 + tf_demo 整合 TF 演示
- 目录重组：cad/ legacy_ros1/ matlab/ standalone/ ros2_ws/
- robotic_sldasm_ros2_humble 改名 robotic_description，作为唯一描述资产包
- mujoco 单一数据源：robotic_arm.xml（平台+臂链+执行器接口）+ robotic_torque.xml
- robotic_tf_demo：scene 顶层 include 臂模型，viewer 桥接发布 /joint_states，
  tf_static.launch.py 整合 robot_state_publisher + RViz，移除关节滑条方案
- README 全部更新为中文，补充常用命令

File: ros2_ws/src/robotic_description/urdf/robotic.urdf (robot description, URDF)
Before this commit: robot robotic_sldasm, 5 links, 4 joints
Links:
- link base_link: geometry collision mesh filename=package://robotic_description/meshes/base_link.STL; visual mesh filename=package://robotic_description/meshes/base_link.STL
- link link1: geometry collision mesh filename=package://robotic_description/meshes/link1.STL; visual mesh filename=package://robotic_description/meshes/link1.STL
- link link2: geometry collision mesh filename=package://robotic_description/meshes/link2.STL; visual mesh filename=package://robotic_description/meshes/link2.STL
- link link3: geometry collision mesh filename=package://robotic_description/meshes/link3.STL; visual mesh filename=package://robotic_description/meshes/link3.STL
- link link4: geometry collision mesh filename=package://robotic_description/meshes/link4.STL; visual mesh filename=package://robotic_description/meshes/link4.STL
